File: PowerBoard_HF2/PowerBoard_HF2.kicad_sch (KiCad schematic)
At the start: 24 parts, among them J1 Power Supply

Commit message: board updates
Parts:
- removed 5REG1: AP63205WU, Package_TO_SOT_SMD:TSOT-23-6, symbol Regulator_Switching:AP63205WU
- added C5: 22uF, symbol Device:C_Small
- added J2: PCIE, symbol PCIE:PCIE-LP-01-01-F-DV-A-TR_(card_edge)
- added R6: 88.7k, symbol Device:R_Small
- added R7: 22.1k, symbol Device:R_Small
- added REG1: TPS560430X3FDBVT, Package_TO_SOT_SMD:SOT-23-6, symbol Regulator_Switching:TPS560430X3FDBVT
- C4: value 100nF -> 0.1uF
- L2: value 4.7uH -> 18
- R1: value 1k -> 10k
- R4, R5: value 100 -> 1k
- renumbered 3.3REG1 to REG2
Connections:
- net 12V: now also C5.2, J2.A16, J2.A17, J2.A18, J2.B16, J2.B17, J2.B18, REG1.4 (EN), REG1.5 (VIN)
- net 3.3V: now also J2.B13, J2.B14
- net 5V: now also J2.A13, J2.A14
- net GND: now also C5.1, J2.A12, J2.A15, J2.A3, J2.A7, J2.B12, J2.B15, J2.B3, J2.B4, J2.B8, R7.2, REG1.2 (GND)
- net at C6.2, D5.2 (A), F2.1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: now also R6.1
- net at C4.1, D5.1 (K), L2.1: now also REG1.6 (SW)
- net at C4.2: now also REG1.1 (CB)
- new net 5FB: R6.2, R7.1, REG1.3 (FB)
- no-connect marks 0 -> 17
Other:
- note added: "Connect to Battery/ Power Supply"
- note added: "PCIE"
- note added: "Voltage Regulators Overcurrent/ Overvoltage Protection"
- moved on the sheet: C1, C2, C3, C4, C6, C7, D1, D2, D3, D4, D5, F1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

Commit message: more smol updates
Parts:
- removed J1: Power Supply, symbol Connector:Conn_01x02_Male
Connections:
- net +12V: now reaches F1.1
Changed lines of the file:
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@@
   (junction (at 138.43 74.93) (diameter 0) (color 0 0 0 0)
   )
-  (junction (at 39.37 34.29) (diameter 0) (color 0 0 0 0)
-  )
   (junction (at 35.56 106.68) (diameter 0) (color 0 0 0 0)
   )
@@
   )
   (junction (at 71.12 81.28) (diameter 0) (color 0 0 0 0)
+  )
+  (junction (at 71.12 68.58) (diameter 0) (color 0 0 0 0)
   )
   (junction (at 60.96 99.06) (diameter 0) (color 0 0 0 0)
@@
     (stroke (width 0) (type default) (color 0 0 0 0))
   )
+  (wire (pts (xy 35.56 29.21) (xy 35.56 27.94))
+    (stroke (width 0) (type default) (color 0 0 0 0))
+  )
   (wire (pts (xy 148.59 38.1) (xy 148.59 40.64))
     (stroke (width 0) (type default) (color 0 0 0 0))
@@
     (stroke (width 0) (type default) (color 0 0 0 0))
   )
-  (wire (pts (xy 39.37 31.75) (xy 39.37 34.29))
-    (stroke (width 0) (type default) (color 0 0 0 0))
-  )
   (wire (pts (xy 161.29 33.02) (xy 161.29 38.1))
     (stroke (width 0) (type default) (color 0 0 0 0))
@@
     (stroke (width 0) (type default) (color 0 0 0 0))
   )
-  (wire (pts (xy 39.37 29.21) (xy 44.45 29.21))
+  (wire (pts (xy 35.56 29.21) (xy 44.45 29.21))
     (stroke (width 0) (type default) (color 0 0 0 0))
   )
@@
     (pin "2")
   )
+  (symbol (lib_id "power:+12V") (at 35.56 27.94 0) (unit 1)
+    (in_bom yes) (on_board yes) (fields_autoplaced)
+    (property "Reference" "#PWR01" (id 0) (at 35.56 31.75 0)
+      (effects (font (size 1.27 1.27)) hide)
+    )
+    (property "Value" "+12V" (id 1) (at 35.56 22.86 0))
+    (property "Footprint" "" (id 2) (at 35.56 27.94 0)
+      (effects (font (size 1.27 1.27)) hide)
+    )
+    (property "Datasheet" "" (id 3) (at 35.56 27.94 0)
+      (effects (font (size 1.27 1.27)) hide)
+    )
+    (pin "1")
+  )
   (symbol (lib_id "power:GND") (at 149.86 88.9 0) (unit 1)
     (in_bom yes) (on_board yes) (fields_autoplaced)
@@
     (pin "6")
   )
-  (symbol (lib_id "power:PWR_FLAG") (at 39.37 34.29 90) (unit 1)
-    (in_bom yes) (on_board yes) (fields_autoplaced)
-    (property "Reference" "#FLG01" (id 0) (at 37.465 34.29 0)
-      (effects (font (size 1.27 1.27)) hide)
-    )
-    (property "Value" "PWR_FLAG" (id 1) (at 35.56 34.2899 90)
-      (effects (font (size 1.27 1.27)) (justify left))
-    )
-    (property "Footprint" "" (id 2) (at 39.37 34.29 0)
-      (effects (font (size 1.27 1.27)) hide)
-    )
-    (property "Datasheet" "~" (id 3) (at 39.37 34.29 0)
-      (effects (font (size 1.27 1.27)) hide)
-    )
-    (pin "1")
-  )
-  (symbol (lib_id "Connector:Conn_01x02_Male") (at 34.29 29.21 0) (unit 1)
-    (in_bom yes) (on_board yes) (fields_autoplaced)
-    (property "Reference" "J1" (id 0) (at 34.925 24.13 0))
-    (property "Value" "Power Supply" (id 1) (at 34.925 26.67 0))
-    (property "Footprint" "" (id 2) (at 34.29 29.21 0)
-      (effects (font (size 1.27 1.27)) hide)
-    )
-    (property "Datasheet" "~" (id 3) (at 34.29 29.21 0)
-      (effects (font (size 1.27 1.27)) hide)
-    )
-    (pin "1")
-    (pin "2")
-  )
   (symbol (lib_id "Device:Polyfuse_Small") (at 166.37 74.93 90) (unit 1)
     (in_bom yes) (on_board yes) (fields_autoplaced)
@@
     (pin "1")
   )
+  (symbol (lib_id "power:PWR_FLAG") (at 71.12 68.58 0) (unit 1)
+    (in_bom yes) (on_board yes) (fields_autoplaced)
+    (property "Reference" "#FLG01" (id 0) (at 71.12 66.675 0)
+      (effects (font (size 1.27 1.27)) hide)
+    )
+    (property "Value" "PWR_FLAG" (id 1) (at 71.12 63.5 0))
+    (property "Footprint" "" (id 2) (at 71.12 68.58 0)
+      (effects (font (size 1.27 1.27)) hide)
+    )
+    (property "Datasheet" "~" (id 3) (at 71.12 68.58 0)
+      (effects (font (size 1.27 1.27)) hide)
+    )
+    (pin "1")
+  )
   (symbol (lib_id "power:GND") (at 148.59 46.99 0) (unit 1)
     (in_bom yes) (on_board yes) (fields_autoplaced)
@@
     )
     (property "Datasheet" "" (id 3) (at 148.59 46.99 0)
-      (effects (font (size 1.27 1.27)) hide)
-    )
-    (pin "1")
-  )
-  (symbol (lib_id "power:GND") (at 39.37 34.29 0) (unit 1)
-    (in_bom yes) (on_board yes) (fields_autoplaced)
-    (property "Reference" "#PWR01" (id 0) (at 39.37 40.64 0)
-      (effects (font (size 1.27 1.27)) hide)
-    )
-    (property "Value" "GND" (id 1) (at 39.37 39.37 0))
-    (property "Footprint" "" (id 2) (at 39.37 34.29 0)
-      (effects (font (size 1.27 1.27)) hide)
-    )
-    (property "Datasheet" "" (id 3) (at 39.37 34.29 0)
       (effects (font (size 1.27 1.27)) hide)
     )
@@
   )
   (symbol_instances
-    (path "/abf472c3-320a-45d5-b443-1dc3c5383a19"
+    (path "/d4c6f9f8-4a4d-406f-81f1-842b53e289cb"
       (reference "#FLG01") (unit 1) (value "PWR_FLAG") (footprint "")
     )
@@
       (reference "#FLG03") (unit 1) (value "PWR_FLAG") (footprint "")
     )
-    (path "/ecd61e2a-ccb4-44bc-a9ab-b604d8218dea"
-      (reference "#PWR01") (unit 1) (value "GND") (footprint "")
+    (path "/94022366-a554-423b-87ca-ba5594b6ec3d"
+      (reference "#PWR01") (unit 1) (value "+12V") (footprint "")
     )
     (path "/7e4c92f0-d7fa-4cc3-8ba9-967123f29c0f"
@@
       (reference "F3") (unit 1) (value "500mA Fuse") (footprint "")
     )
-    (path "/b63623f6-c7e7-4d5b-854b-dfe353a57aa0"
-      (reference "J1") (unit 1) (value "Power Supply") (footprint "")
-    )
     (path "/5f96967f-97fe-4ee7-8850-74584e757101"
