File: HX-board/HX-board.kicad_pcb (KiCad board)
At the start: 2 copper layers, 63.5 x 63.9 mm, 101 parts, among them J1 Testpoints, J2 PCIE-LP-01-01-F-DV-A-TR, J3 DB15_Female, J4 Testpoints, J5 DB15_Female, Q1 MMBT4403LT3G, Q2 MMBT4403LT3G, Q3 MMBT4403LT3G, Q4 MMBT4403LT3G, Q5 MMBT4403LT3G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

Commit message: HX and TC Done
Routing:
- net /HX_CLK: track 157.9 -> 155.6 mm
- net GND: track 697.2 -> 695.7 mm
- net /HX711 1/A+: track 16.1 -> 14.7 mm
- net /HX2_E+: track 56.0 -> 56.8 mm
- net /HX1_A+: track 104.5 -> 103.9 mm
- net /HX1_E+: track 98.3 -> 97.7 mm
- added copper zone on F.Cu, net GND
