File: HX-board/HX711_breakout.kicad_sch (KiCad schematic)
At the start: 10 parts, among them Q1 MMBT4403LT3G, U1 HX711

Commit message: Progress on revising ground boards.
Connections:
- net +3.3V: now also U1.15 (RATE)
- net GND: no longer U1.15 (RATE)
Changed lines of the file:
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@@
   (junction (at 103.7059 52.832) (diameter 0) (color 0 0 0 0)
-  )
-  (junction (at 132.588 73.152) (diameter 0) (color 0 0 0 0)
   )
   (junction (at 104.394 83.312) (diameter 0) (color 0 0 0 0)
@@
     (stroke (width 0) (type default) (color 0 0 0 0))
   )
-  (wire (pts (xy 130.81 73.152) (xy 132.588 73.152))
+  (wire (pts (xy 130.81 73.152) (xy 138.176 73.152))
     (stroke (width 0) (type default) (color 0 0 0 0))
   )
@@
   )
   (wire (pts (xy 96.52 65.532) (xy 96.52 83.82))
-    (stroke (width 0) (type default) (color 0 0 0 0))
-  )
-  (wire (pts (xy 132.588 65.532) (xy 132.588 73.152))
     (stroke (width 0) (type default) (color 0 0 0 0))
   )
@@
     (pin "1")
     (pin "2")
+  )
+  (symbol (lib_id "power:+3.3V") (at 138.176 73.152 0) (unit 1)
+    (in_bom yes) (on_board yes)
+    (property "Reference" "#PWR?" (id 0) (at 138.176 76.962 0)
+      (effects (font (size 1.27 1.27)) hide)
+    )
+    (property "Value" "+3.3V" (id 1) (at 137.922 69.342 0))
+    (property "Footprint" "" (id 2) (at 138.176 73.152 0)
+      (effects (font (size 1.27 1.27)) hide)
+    )
+    (property "Datasheet" "" (id 3) (at 138.176 73.152 0)
+      (effects (font (size 1.27 1.27)) hide)
+    )
+    (pin "1")
   )
   (symbol (lib_id "power:+3.3V") (at 120.65 40.132 0) (unit 1)
@@
     (pin "9")
   )
-  (symbol (lib_id "power:GND") (at 132.588 73.152 0) (unit 1)
-    (in_bom yes) (on_board yes)
-    (property "Reference" "#PWR010" (id 0) (at 132.588 79.502 0)
-      (effects (font (size 1.27 1.27)) hide)
-    )
-    (property "Value" "GND" (id 1) (at 132.588 77.216 0))
-    (property "Footprint" "" (id 2) (at 132.588 73.152 0)
-      (effects (font (size 1.27 1.27)) hide)
-    )
-    (property "Datasheet" "" (id 3) (at 132.588 73.152 0)
-      (effects (font (size 1.27 1.27)) hide)
-    )
+  (symbol (lib_id "power:GND") (at 132.588 65.532 0) (unit 1)
+    (in_bom yes) (on_board yes)
+    (property "Reference" "#PWR010" (id 0) (at 132.588 71.882 0)
+      (effects (font (size 1.27 1.27)) hide)
+    )
+    (property "Value" "GND" (id 1) (at 132.588 69.596 0))
+    (property "Footprint" "" (id 2) (at 132.588 65.532 0)
+      (effects (font (size 1.27 1.27)) hide)
+    )
+    (property "Datasheet" "" (id 3) (at 132.588 65.532 0)
+      (effects (font (size 1.27 1.27)) hide)
+    )
