File: Core-Board/Core-Board.kicad_sch (KiCad schematic)
At the start: 37 parts, among them J1 POWER, J10 PCIE, J2 PCIE, J3 XT60-M, J4 PCIE, J5 PCIE, J6 ESP32-DEVKITC-32D, J7 Conn_01x19_Male, J8 PCIE, J9 Conn_01x19_Male, SW1 SW_SPST, U1 AZ1117IH-3.3TRG1, U2 74HC4050D, U3 XTSD04GLGEAG, U4 AZ1117IH-5TRG1

Commit message: Revising PCIe.
Parts:
- removed J10, J2, J4, J5, J8: PCIE, 10018784-10210TLF:AMPHENOL_10018784-10210TLF, symbol PCIE:PCIE-LP-01-01-F-DV-A-TR_(card_edge)
- removed U?: MCP23S17-E_SO, MCP23S17-E_SO:SOIC127P1030X265-28N, symbol MCP23S17-E_SO:MCP23S17-E_SO
- added J? (x2): PCIE-164-02-X-D-TH, PCIE-164-02-X-D-TH:SAMTEC_PCIE-164-02-X-D-TH, symbol PCIE-164-02-X-D-TH:PCIE-164-02-X-D-TH
- added U?: PCF8575DW, PCF8575DW:SOIC127P1030X265-24N, symbol PCF8575DW:PCF8575DW
Connections:
- net 3.3V: now also J?.A20, J?.A21, J?.A22, J?.A23, J?.B20, J?.B21, J?.B22, J?.B23, U?.24 (VCC)
- net 5V: now also J?.A14, J?.A15, J?.A16, J?.A17, J?.B14, J?.B15, J?.B16, J?.B17
- net BAT2_+: now also J?.A1, J?.A2, J?.A3, J?.A4, J?.A5, J?.B1, J?.B2, J?.B3, J?.B4, J?.B5
- net BAT2_-: now also J?.A10, J?.A11, J?.A6, J?.A7, J?.A8, J?.A9, J?.B10, J?.B11, J?.B6, J?.B7, J?.B8, J?.B9
- net GND: now also J?.A12, J?.A13, J?.A18, J?.A19, J?.A24, J?.A25, J?.A27, J?.A29, J?.A31, J?.A33, J?.A35, J?.A37, J?.A39, J?.A41, J?.A43, J?.A45, J?.A47, J?.B12, J?.B13, J?.B18, J?.B19, J?.B24, J?.B25, J?.B27, J?.B29, J?.B31, J?.B33, J?.B35, J?.B37, J?.B39, J?.B41, J?.B43, J?.B45, J?.B47, U?.12 (GND), U?.2 (A1), U?.21 (A0), U?.3 (A2)
- net HX CLK: now also J?.A46
- net HX1: now also J?.A30
- net HX2: now also J?.A32
- net HX3: now also J?.A34
- net HX4: now also J?.A36
- net HX5: now also J?.A38
- net HX6: now also J?.A40
- net HX7: now also J?.A42
- net HX8: now also J?.A44
- net MOS SCL: now also J?.A28
- net MOS SDA: now also J?.A26
- net TC CLK: now also J?.B26
- net TC MISO: now also J?.B28
- net TC MOSI: now also J6.30 (IO17), J?.B30
- net TC1: no longer J6.30 (IO17)
- net TC2: no longer J6.31 (IO16)
- net TC3: no longer J6.32 (IO4)
- net TC4: no longer J6.35 (IO15)
- new net CS1: J?.B32, U?.4 (P00)
- new net CS2: J?.B34, U?.5 (P01)
- new net CS3: J?.B36, U?.6 (P02)
- new net CS4: J?.B38, U?.7 (P03)
- new net CS5: J?.B40, U?.8 (P04)
- new net CS6: J?.B42, U?.9 (P05)
- new net CS7: J?.B44, U?.10 (P06)
- new net CS8: J?.B46, U?.11 (P07)
- new net I2C SCL: U?.22 (SCL)
- new net I2C SDA: U?.23 (SDA)
- new net SERIAL_RX: J6.31 (IO16)
- new net SERIAL_TX: J6.32 (IO4)
- no-connect marks 38 -> 115

Commit message: Ironing out small details, changed pcf8575 to IC instead of breakout.
Parts:
- removed C?: 22uF, Capacitor_SMD:C_0603_1608Metric, symbol Device:C_Small
- removed D?: D_Small, Diode_SMD:D_0603_1608Metric, symbol Device:D_Small
- removed F?: 6A Fuse, Fuse:Fuse_2920_7451Metric, symbol Device:Polyfuse_Small
- removed R?: 10k, Resistor_SMD:R_0603_1608Metric, symbol Device:R_Small
- added C6: 22uF, Capacitor_SMD:C_0603_1608Metric, symbol Device:C_Small
- added D2: D_Small, Diode_SMD:D_0603_1608Metric, symbol Device:D_Small
- added F1: 6A Fuse, Fuse:Fuse_2920_7451Metric, symbol Device:Polyfuse_Small
- added J13: Conn_01x08_Male, Connector_PinHeader_2.54mm:PinHeader_1x08_P2.54mm_Vertical, symbol Connector:Conn_01x08_Male
- added J14, J15, J16, J17: PCIE-164-02-X-D-TH, PCIE-164-02-X-D-TH:SAMTEC_PCIE-164-02-X-D-TH, symbol PCIE-164-02-X-D-TH:PCIE-164-02-X-D-TH
- added J18, J19, J20: Conn_01x02_Male, Connector_PinHeader_2.54mm:PinHeader_1x02_P2.54mm_Vertical, symbol Connector:Conn_01x02_Male
- added R3, R4, R5, R6: 10k, Resistor_SMD:R_0603_1608Metric, symbol Device:R_Small
- J10, J2: renamed from J?; footprint (none) -> Connector_PinHeader_2.54mm:PinHeader_1x02_P2.54mm_Vertical
- J12: renamed from J?; footprint (none) -> DSUB_622-015-260-042:DSUB_622-015-260-042
- gave numbers to parts that had none: 5
Connections:
- net BAT1_+ is gone; now on net 12V: J12.11 (P111), J12.4
- net BAT1_- is gone; now on net GND: J12.10 (P10), J12.2, J12.3
- net MOS SCL is gone; now on net I2C SCL: J11.A28, J6.22 (IO22), J9.3 (Pin_3)
- net MOS SDA is gone; now on net I2C SDA: J11.A26, J6.25 (IO21), J9.6 (Pin_6)
- net Serial_RX is gone; now on net SERIAL_RX: J12.1
- net Serial_TX is gone; now on net SERIAL_TX: J12.9 (P9)
- net TC1 is gone; now on net TC MOSI: J9.11 (Pin_11)
- net TC2 is gone; now on net SERIAL_RX: J9.12 (Pin_12)
- net TC3 is gone; now on net SERIAL_TX: J9.13 (Pin_13)
- net +12V: no longer J5.1 (Pin_1), J8.P (POS)
- net +3.3V: no longer J7.19 (Pin_19)
- net +5V: no longer J7.1 (Pin_1)
- net 12V: now also F1.2
- net 3.3V: now also J7.19 (Pin_19), J14.A20, J14.A21, J14.A22, J14.A23, J14.B20, J14.B21, J14.B22, J14.B23, J15.A20, J15.A21, J15.A22, J15.A23, J15.B20, J15.B21, J15.B22, J15.B23, J16.A20, J16.A21, J16.A22, J16.A23, J16.B20, J16.B21, J16.B22, J16.B23, J17.A20, J17.A21, J17.A22, J17.A23, J17.B20, J17.B21, J17.B22, J17.B23, J18.1 (Pin_1), J19.1 (Pin_1), J20.1 (Pin_1)
- net 5V: now also J7.1 (Pin_1), J14.A14, J14.A15, J14.A16, J14.A17, J14.B14, J14.B15, J14.B16, J14.B17, J15.A14, J15.A15, J15.A16, J15.A17, J15.B14, J15.B15, J15.B16, J15.B17, J16.A14, J16.A15, J16.A16, J16.A17, J16.B14, J16.B15, J16.B16, J16.B17, J17.A14, J17.A15, J17.A16, J17.A17, J17.B14, J17.B15, J17.B16, J17.B17
- net BAT2_+: now also J14.A1, J14.A2, J14.A3, J14.A4, J14.A5, J14.B1, J14.B2, J14.B3, J14.B4, J14.B5, J15.A1, J15.A2, J15.A3, J15.A4, J15.A5, J15.B1, J15.B2, J15.B3, J15.B4, J15.B5, J16.A1, J16.A2, J16.A3, J16.A4, J16.A5, J16.B1, J16.B2, J16.B3, J16.B4, J16.B5, J17.A1, J17.A2, J17.A3, J17.A4, J17.A5, J17.B1, J17.B2, J17.B3, J17.B4, J17.B5
- net BAT2_-: now also J14.A10, J14.A11, J14.A6, J14.A7, J14.A8, J14.A9, J14.B10, J14.B11, J14.B6, J14.B7, J14.B8, J14.B9, J15.A10, J15.A11, J15.A6, J15.A7, J15.A8, J15.A9, J15.B10, J15.B11, J15.B6, J15.B7, J15.B8, J15.B9, J16.A10, J16.A11, J16.A6, J16.A7, J16.A8, J16.A9, J16.B10, J16.B11, J16.B6, J16.B7, J16.B8, J16.B9, J17.A10, J17.A11, J17.A6, J17.A7, J17.A8, J17.A9, J17.B10, J17.B11, J17.B6, J17.B7, J17.B8, J17.B9
- net CS1: now also J13.1 (Pin_1), J14.B32, J15.B32, J16.B32, J17.B32
- net CS2: now also J13.2 (Pin_2), J14.B34, J15.B34, J16.B34, J17.B34
- net CS3: now also J13.3 (Pin_3), J14.B36, J15.B36, J16.B36, J17.B36
- net CS4: now also J13.4 (Pin_4), J14.B38, J15.B38, J16.B38, J17.B38
- net CS5: now also J13.5 (Pin_5), J14.B40, J15.B40, J16.B40, J17.B40
- net CS6: now also J13.6 (Pin_6), J14.B42, J15.B42, J16.B42, J17.B42
- net CS7: now also J13.7 (Pin_7), J14.B44, J15.B44, J16.B44, J17.B44
- net CS8: now also J13.8 (Pin_8), J14.B46, J15.B46, J16.B46, J17.B46
- net GND: now also C6.1, D2.2 (A), J14.A12, J14.A13, J14.A18, J14.A19, J14.A24, J14.A25, J14.A27, J14.A29, J14.A31, J14.A33, J14.A35, J14.A37, J14.A39, J14.A41, J14.A43, J14.A45, J14.A47, J14.B12, J14.B13, J14.B18, J14.B19, J14.B24, J14.B25, J14.B27, J14.B29, J14.B31, J14.B33, J14.B35, J14.B37, J14.B39, J14.B41, J14.B43, J14.B45, J14.B47, J15.A12, J15.A13, J15.A18, J15.A19, J15.A24, J15.A25, J15.A27, J15.A29, J15.A31, J15.A33, J15.A35, J15.A37, J15.A39, J15.A41, J15.A43, J15.A45, J15.A47, J15.B12, J15.B13, J15.B18, J15.B19, J15.B24, J15.B25, J15.B27, J15.B29, J15.B31, J15.B33, J15.B35, J15.B37, J15.B39, J15.B41, J15.B43, J15.B45, J15.B47, J16.A12, J16.A13, J16.A18, J16.A19, J16.A24, J16.A25, J16.A27, J16.A29, J16.A31, J16.A33, J16.A35, J16.A37, J16.A39, J16.A41, J16.A43, J16.A45, J16.A47, J16.B12, J16.B13, J16.B18, J16.B19, J16.B24, J16.B25, J16.B27, J16.B29, J16.B31, J16.B33, J16.B35, J16.B37, J16.B39, J16.B41, J16.B43, J16.B45, J16.B47, J17.A12, J17.A13, J17.A18, J17.A19, J17.A24, J17.A25, J17.A27, J17.A29, J17.A31, J17.A33, J17.A35, J17.A37, J17.A39, J17.A41, J17.A43, J17.A45, J17.A47, J17.B12, J17.B13, J17.B18, J17.B19, J17.B24, J17.B25, J17.B27, J17.B29, J17.B31, J17.B33, J17.B35, J17.B37, J17.B39, J17.B41, J17.B43, J17.B45, J17.B47, R4.1, R5.1, R6.1; no longer U5.2 (A1), U5.21 (A0), U5.3 (A2)
- net HX CLK: now also J14.A46, J15.A46, J16.A46, J17.A46
- net HX1: now also J14.A30, J15.A30, J16.A30, J17.A30
- net HX2: now also J14.A32, J15.A32, J16.A32, J17.A32
- net HX3: now also J14.A34, J15.A34, J16.A34, J17.A34
- net HX4: now also J14.A36, J15.A36, J16.A36, J17.A36
- net HX5: now also J14.A38, J15.A38, J16.A38, J17.A38
- net HX6: now also J14.A40, J15.A40, J16.A40, J17.A40
- net HX7: now also J14.A42, J15.A42, J16.A42, J17.A42
- net HX8: now also J14.A44, J15.A44, J16.A44, J17.A44
- net I2C SCL: now also J14.A28, J15.A28, J16.A28, J17.A28
- net I2C SDA: now also J14.A26, J15.A26, J16.A26, J17.A26
- net TC CLK: now also J14.B26, J15.B26, J16.B26, J17.B26
- net TC MISO: now also J14.B28, J15.B28, J16.B28, J17.B28
- net TC MOSI: now also J14.B30, J15.B30, J16.B30, J17.B30
- net SD, TC CLK renamed SD CLK
- net SD, TC MISO renamed SD MISO
- net TC4: no longer names the net of J9.16 (Pin_16)
- new net: J20.2 (Pin_2), R6.2, U5.3 (A2)
- new net: D2.1 (K), R3.2
- new net: J19.2 (Pin_2), R5.2, U5.2 (A1)
- new net: J18.2 (Pin_2), R4.2, U5.21 (A0)
- new net BAT1_+_pre: C6.2, F1.1, J5.1 (Pin_1), J8.P (POS), R3.1
- no-connect marks 115 -> 396
Other:
- moved on the sheet: J11A, J11B, J12, U5
