File: MOSFET-board/i2c_level_shifter.kicad_sch (KiCad schematic)
At the start: 8 parts, among them J4 Pin Jumper, J5 Pin Jumper, Q1 NMOS, Q2 NMOS

Commit message: Ironing out small details, changed pcf8575 to IC instead of breakout.
Parts:
- J4, J5: footprint (none) -> Connector_PinHeader_2.54mm:PinHeader_1x02_P2.54mm_Vertical
- R1, R2, R5, R6: footprint (none) -> Resistor_SMD:R_0603_1608Metric
Changed lines of the file:
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@@
       (effects (font (size 1.27 1.27)) (justify left))
     )
-    (property "Footprint" "" (at 108.712 125.984 0)
+    (property "Footprint" "Resistor_SMD:R_0603_1608Metric" (at 108.712 125.984 0)
       (effects (font (size 1.27 1.27)) hide)
     )
@@
       (effects (font (size 1.27 1.27)) (justify left))
     )
-    (property "Footprint" "" (at 108.966 100.33 0)
+    (property "Footprint" "Resistor_SMD:R_0603_1608Metric" (at 108.966 100.33 0)
       (effects (font (size 1.27 1.27)) hide)
     )
@@
       (effects (font (size 1.27 1.27)) (justify left))
     )
-    (property "Footprint" "" (at 125.222 125.984 0)
+    (property "Footprint" "Resistor_SMD:R_0603_1608Metric" (at 125.222 125.984 0)
       (effects (font (size 1.27 1.27)) hide)
     )
@@
       (effects (font (size 1.27 1.27)) (justify right))
     )
-    (property "Footprint" "" (at 157.734 101.092 0)
+    (property "Footprint" "Connector_PinHeader_2.54mm:PinHeader_1x02_P2.54mm_Vertical" (at 157.734 101.092 0)
       (effects (font (size 1.27 1.27)) hide)
     )
@@
       (effects (font (size 1.27 1.27)) (justify left))
     )
-    (property "Footprint" "" (at 125.476 100.33 0)
+    (property "Footprint" "Resistor_SMD:R_0603_1608Metric" (at 125.476 100.33 0)
       (effects (font (size 1.27 1.27)) hide)
     )
@@
       (effects (font (size 1.27 1.27)) (justify right))
     )
-    (property "Footprint" "" (at 157.48 124.968 0)
+    (property "Footprint" "Connector_PinHeader_2.54mm:PinHeader_1x02_P2.54mm_Vertical" (at 157.48 124.968 0)
       (effects (font (size 1.27 1.27)) hide)
     )
