File: MOSFET-board/pyro.kicad_sch (KiCad schematic)
At the start: 11 parts, among them U1 BTS3080EJXUMA1, U19 INA193

Commit message: MOSFET Board Updated (Part IV? I lost count)
Has a specified op amp, fixed measurements, should be a double header GPIO, I believe that everything is connected. The only warnings are either silk screen or non labeled items, which should be fine.
Parts:
- removed U19: INA193, Package_TO_SOT_SMD:SOT-23-5, symbol Amplifier_Current:INA193
- added U24: ADA4897-1ARJZ-R7, Symbol:SOT95P280X145-6N, symbol Amplifier_Operational:ADA4897-1ARJZ-R7
Connections:
- net +5V: now also U24.6
- net GND: now also U24.2
- net In: now also U24.3
- net at R103.2, R83.1, R93.1: now also U24.1
- net at R73.1, R83.2: now also U24.4
- no-connect marks 1 -> 2
