File: flight-module/Power-board/pyro.kicad_sch (KiCad schematic)
At the start: 7 parts, among them Q1 Q_PMOS_GDS

Commit message: changed to one battery
Connections:
- net V_pyro_+ renamed SENS_N_PYRO+
Changed lines of the file:
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@@
     (stroke (width 0) (type default))
   )
-  (global_label "V_pyro_+" (shape input) (at 89.916 43.18 0) (fields_autoplaced)
+  (global_label "SENS_N_PYRO+" (shape input) (at 89.916 43.18 0) (fields_autoplaced)
     (effects (font (size 1.27 1.27)) (justify left))
-    (property "Intersheetrefs" "${INTERSHEET_REFS}" (at 101.5492 43.18 0)
+    (property "Intersheetrefs" "${INTERSHEET_REFS}" (at 107.5969 43.18 0)
       (effects (font (size 1.27 1.27)) (justify left) hide)
     )
