File: flight-module/Power-board/Power-board.kicad_pcb (KiCad board)
At the start: 4 copper layers, 141.7 x 134.1 mm, 48 parts, among them J1 Stack_Shape, J2 XT60-M, J5 POWER, U1 AZ1117IH-3.3TRG1, U2 TPS4H160BQPWPRQ1, U3 TPS4H160BQPWPRQ1, U4 AZ1117IH-5TRG1

Commit message: fixed all errors
Parts:
- moved G*** 17.3 mm to (122.9, 114.6)
- moved C9 0.38 mm to (116.5, 74.2)
- moved D8 0.38 mm to (112.4, 74.2)
Routing:
- net GND: track 77.4 -> 83.7 mm, vias 28 -> 29
- net ETH_VENT+: track 78.4 -> 75.7 mm
- net ETH_MAIN+: track 56.3 -> 54.0 mm
- net V_ALL+: vias 28 -> 38

Commit message: not done just commiting just in case
Parts:
- added R10: 1, Resistor_SMD:R_0603_1608Metric, F.Cu at (125.2, 90.9)
- added R7: 1, Resistor_SMD:R_0603_1608Metric, F.Cu at (125.3, 81.3)
- added R8: 1, Resistor_SMD:R_0603_1608Metric, F.Cu at (125.2, 84.3)
- added R9: 1, Resistor_SMD:R_0603_1608Metric, F.Cu at (125.2, 87.6)
- R2, R4, R5, R6: value 2k -> 100
- moved D4 6.81 mm to (133.8, 87.6)
- moved D3 6.81 mm to (133.8, 84.3)
- moved D1 6.81 mm to (133.7, 78.0)
- moved D5 6.81 mm to (133.8, 93.5)
- moved R5 6.81 mm to (129.0, 87.6)
- moved R2 6.81 mm to (129.0, 81.2)
- moved R4 6.81 mm to (129.0, 84.3)
- moved R6 6.81 mm to (129.0, 90.9)
- moved C6 5.66 mm to (154.3, 83.6)
- moved D15 5.66 mm to (162.8, 96.6)
- moved C11 5.66 mm to (149.6, 93.4)
- moved C12 5.66 mm to (158.0, 93.6)
- moved C7 5.66 mm to (162.6, 102.2)
- moved D2 5.66 mm to (149.1, 86.1)
- moved F1 5.66 mm to (162.2, 84.7)
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Connections:
- U2 pad 11: unconnected-(U2-CL-Pad11) -> GND
- U3 pad 11: unconnected-(U3-CL-Pad11) -> GND
Routing:
- net PYRO_EX+: track 78.3 -> 86.3 mm
- net ETH_MAIN+: track 54.0 -> 61.6 mm
- net ETH_VENT+: track 75.7 -> 83.3 mm
- net LOX_VENT+: track 75.5 -> 82.5 mm
- net GND: track 83.7 -> 89.7 mm, vias 29 -> 33
- net /BAT1_+_pre: track 83.7 -> 82.3 mm
- net PYRO4EN: track 130.9 -> 131.6 mm
- net V_ALL+: vias 38 -> 37

Commit message: more updates to flight power
Parts:
- moved D10 0.28 mm to (112.5, 81.8)
Routing:
- net PYRO_EX+: track 86.3 -> 83.1 mm
- net ETH_MAIN+: track 61.6 -> 63.7 mm
- net ETH_VENT+: track 83.3 -> 84.8 mm
- net LOX_VENT+: track 82.5 -> 81.2 mm

Commit message: board review updates done
Parts:
- added D14: D_Small, Diode_SMD:D_0603_1608Metric, F.Cu at (130.0, 68.6)
- added D17: D_Small, Diode_SMD:D_0603_1608Metric, F.Cu at (125.0, 68.5)
- added D18: D_Small, Diode_SMD:D_0603_1608Metric, F.Cu at (125.0, 70.6)
- added D19: D_Small, Diode_SMD:D_0603_1608Metric, F.Cu at (125.0, 72.9)
- added D20: D_Small, Diode_SMD:D_0603_1608Metric, F.Cu at (125.0, 75.2)
- added D21: D_Small, Diode_SMD:D_0603_1608Metric, F.Cu at (130.1, 72.9)
- added D22: D_Small, Diode_SMD:D_0603_1608Metric, F.Cu at (130.1, 70.7)
- added D23: D_Small, Diode_SMD:D_0603_1608Metric, F.Cu at (130.1, 75.3)
- added JP1: SolderJumper_2_Open, Jumper:SolderJumper-2_P1.3mm_Bridged_RoundedPad1.0x1.5mm, F.Cu at (97.6, 66.8)
- added JP2: SolderJumper_2_Open, Jumper:SolderJumper-2_P1.3mm_Bridged_RoundedPad1.0x1.5mm, F.Cu at (97.6, 69.6)
- added JP3: SolderJumper_2_Open, Jumper:SolderJumper-2_P1.3mm_Bridged_RoundedPad1.0x1.5mm, F.Cu at (97.6, 72.4)
- added JP4: SolderJumper_2_Open, Jumper:SolderJumper-2_P1.3mm_Bridged_RoundedPad1.0x1.5mm, F.Cu at (97.6, 75.2)
- added JP5: SolderJumper_2_Open, Jumper:SolderJumper-2_P1.3mm_Bridged_RoundedPad1.0x1.5mm, F.Cu at (97.4, 82.3)
- added JP6: SolderJumper_2_Open, Jumper:SolderJumper-2_P1.3mm_Bridged_RoundedPad1.0x1.5mm, F.Cu at (97.4, 85.1)
- added JP7: SolderJumper_2_Open, Jumper:SolderJumper-2_P1.3mm_Bridged_RoundedPad1.0x1.5mm, F.Cu at (97.4, 87.9)
- added JP8: SolderJumper_2_Open, Jumper:SolderJumper-2_P1.3mm_Bridged_RoundedPad1.0x1.5mm, F.Cu at (97.4, 90.7)
- R10, R7, R8, R9: value 1 -> 1k
- R2, R4, R5, R6: value 100 -> 100k
- moved D12 6.65 mm to (112.3, 84.1)
- moved C15 4.61 mm to (116.1, 84.1)
- moved D11 4.55 mm to (112.8, 88.6)
- moved C14 4.55 mm to (116.3, 88.6)
- moved D13 2.00 mm to (112.8, 90.7)
- moved C16 0.09 mm to (116.3, 90.8)
- moved J1 0.09 mm to (123.2, 86.0)
Connections:
- C14 pad 1: ETH_VENT+ -> ETH_MAIIN+
- C15 pad 1: ETH_MAIIN+ -> ETH_VENT+
- D11 pad 1: ETH_VENT+ -> ETH_MAIIN+
- D12 pad 1: PYRO_EX+ -> ETH_VENT+
- D13 pad 1: ETH_MAIIN+ -> PYRO_EX+
- U2 pad 15: Net-(D12-A) -> Net-(D13-A)
- U2 pad 16: Net-(D12-A) -> Net-(D13-A)
- U2 pad 17: Net-(D13-A) -> Net-(D11-A)
- U2 pad 18: Net-(D13-A) -> Net-(D11-A)
- U2 pad 25: Net-(D11-A) -> Net-(D12-A)
- U2 pad 26: Net-(D11-A) -> Net-(D12-A)
- U2 pad 3: PYRO1EN -> Net-(JP5-B)
- U2 pad 4: PYRO2EN -> Net-(JP6-B)
- U2 pad 5: PYRO3EN -> Net-(JP7-B)
- U2 pad 6: PYRO4EN -> Net-(JP8-B)
- U3 pad 3: PYRO1EN -> Net-(JP1-B)
- U3 pad 4: PYRO2EN -> Net-(JP2-B)
- U3 pad 5: PYRO3EN -> Net-(JP3-B)
- U3 pad 6: PYRO4EN -> Net-(JP4-B)
Routing:
- net PYRO_EX+: track 83.1 -> 103.5 mm
- net LOX_VENT+: track 81.2 -> 97.7 mm
- net ETH_MAIIN+: track 20.5 -> 35.9 mm
- net GND: track 89.7 -> 102.8 mm, vias 33 -> 41
- net ETH_VENT+: track 84.8 -> 97.6 mm
- net Net-(JP8-B): track 0.00 -> 7.81 mm
- net PYRO4EN: track 131.6 -> 138.5 mm, vias 2 -> 0
- net Net-(JP4-B): track 0.00 -> 6.89 mm
- net Net-(JP7-B): track 0.00 -> 6.13 mm
- net Net-(JP3-B): track 0.00 -> 5.56 mm
- net Net-(JP1-B): track 0.00 -> 5.49 mm
- net Net-(JP5-B): track 0.00 -> 5.32 mm
- net Net-(JP6-B): track 0.00 -> 5.24 mm
- net PYRO3EN: track 124.9 -> 129.8 mm
- net Net-(JP2-B): track 0.00 -> 4.73 mm
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Other:
- board text added: "+"
- board text added: "-"
