File: flight-module/Connector-board/Connector-board.kicad_sch (KiCad schematic)
At the start: 15 parts, among them J1 Stack_Shape, J2 DB15_Female, J3 DB15_Female, J4 DB15_Female, J5 DB15_Female

Commit message: Commit changes to the Connector
Parts:
- removed J3, J4, J5: DB15_Female, symbol Connector:DB15_Female
- added J1, J3: DB9_Female, Connector_Dsub:DSUB-9_Female_Vertical_P2.77x2.84mm_MountingHoles, symbol Connector:DE9_Receptacle
- added J5: DB25_Receptacle, Connector_Dsub:DSUB-25_Male_Vertical_P2.77x2.84mm_MountingHoles, symbol Connector:DB25_Receptacle
- C1: renamed from C10; footprint (none) -> Diode_SMD:D_0603_1608Metric
- C2: renamed from C9; footprint (none) -> Diode_SMD:D_0603_1608Metric
- D1: renamed from D9; footprint (none) -> Diode_SMD:D_0603_1608Metric
- D2: renamed from D11; footprint (none) -> Diode_SMD:D_0603_1608Metric
- D3: renamed from D10; footprint (none) -> Diode_SMD:D_0603_1608Metric
- D4: renamed from D1; footprint (none) -> Diode_SMD:D_0603_1608Metric
- D5: renamed from D2; footprint (none) -> Diode_SMD:D_0603_1608Metric
- D6: renamed from D3; footprint (none) -> Diode_SMD:D_0603_1608Metric
- J4: renamed from J2; footprint (none) -> Connector_Dsub:DSUB-15_Female_Vertical_P2.77x2.84mm_MountingHoles
- R1: renamed from R10; footprint (none) -> Diode_SMD:D_0603_1608Metric
- R2: renamed from R5; footprint (none) -> Diode_SMD:D_0603_1608Metric
- renumbered J1 to J2
Connections:
- net PWR SUP 2- is gone; now on net GND: J2.A3 (Pin_3), J2.A4 (Pin_4)
- net +3.3V: no longer J2.A1 (Pin_1), J2.A2 (Pin_2)
- net +5V: now also J2.A5 (Pin_5), J2.A6 (Pin_6), J2.A7 (Pin_7), J2.A8 (Pin_8)
- net Flight_ETH_Vent: no longer J2.A15 (Pin_15), J2.A16 (Pin_16)
- net Flight_LOX_Vent: no longer J2.A11 (Pin_11), J2.A12 (Pin_12)
- net GND: now also J2.A10 (Pin_10), J2.A13 (Pin_13), J2.A14 (Pin_14), J2.A17 (Pin_17), J2.A18 (Pin_18), J2.A22 (Pin_22), J2.A25 (Pin_25), J2.A26 (Pin_26), J2.A9 (Pin_9), J4.10 (P10), J4.11 (P111), J1.6, J1.7; no longer J2.B17 (Pin_17), J2.B25 (Pin_25), J2.B5 (Pin_5), J2.B9 (Pin_9)
- net GND2: no longer J2.A10 (Pin_10), J2.A13 (Pin_13), J2.A14 (Pin_14), J2.A17 (Pin_17), J2.A18 (Pin_18), J2.A21 (Pin_21), J2.A22 (Pin_22), J2.A25 (Pin_25), J2.A26 (Pin_26), J2.A33 (Pin_33), J2.A34 (Pin_34), J2.A9 (Pin_9), J4.10 (P10), J4.11 (P111), J4.12 (P12)
- net Ground_ETH_Vent: no longer J4.5
- net Ground_LOX_Vent: no longer J4.6
- net PT1_A+: now also J5.14 (P14)
- net PT1_E+: now also J5.1
- net PT1_E-: now also J5.2
- net PT2_A+: now also J5.16 (P16)
- net PT2_E+: now also J5.3
- net PT2_E-: now also J5.15 (P15)
- net PT3_A+: now also J5.17 (P17)
- net PT3_E+: now also J5.4
- net PT3_E-: now also J5.5
- net PT4_A+: now also J5.19 (P19); no longer J2.B39 (Pin_39)
- net PT4_E+: now also J2.B37 (Pin_37), J5.6
- net PT4_E-: now also J5.18 (P18); no longer J2.B37 (Pin_37)
- net PT5_A+: now also J5.20 (P20)
- net PT5_E+: now also J5.7
- net PT5_E-: now also J5.8
- net PT6_A+: now also J5.9
- net PT6_E+: now also J5.21 (P21)
- net PT6_E-: now also J5.22 (P22)
- net REDS_ETH_Vent: no longer J4.13 (P13)
- net REDS_LOX_Vent: no longer J4.14 (P14)
- net SPI1_MISO: no longer J2.B4 (Pin_4)
- net SPI1_SCK: no longer J2.B2 (Pin_2)
- net TC1_T+: now also J3.6
- net TC1_T-: now also J3.1
- net TC2_T+: now also J3.7
- net TC2_T-: now also J3.2
- net TC3_T+: now also J3.8
- net TC3_T-: now also J3.3
- net TC4_T+: now also J3.9
- net TC4_T-: now also J3.4
- net I2C_SDA: now reaches J2.B1 (Pin_1)
- net EX_2: now reaches J2.B22 (Pin_22)
- net EX_3: now reaches J2.B24 (Pin_24)
- net I2C_SCL: now reaches J2.B3 (Pin_3)
- net FSPI_MOSI: now reaches J2.B6 (Pin_6)
- net EX_1: now reaches J2.B7 (Pin_7)
- removed net PWR SUP 1+: J2.A27 (Pin_27), J2.A28 (Pin_28), J2.A29 (Pin_29), J2.A30 (Pin_30), J2.A31 (Pin_31), J2.A32 (Pin_32), J4.1
- net PWR SUP 2+ renamed PWR_SUP
- net PWR_SUP: now also J4.1; no longer J2.A35 (Pin_35), J2.A37 (Pin_37), J2.A39 (Pin_39)
- new net: J2.A35 (Pin_35), J2.A37 (Pin_37), J2.A39 (Pin_39)
- new net: J2.B17 (Pin_17), J2.B5 (Pin_5), J2.B9 (Pin_9)
- new net +3V3: J2.A1 (Pin_1), J2.A2 (Pin_2)
- new net ETH_VENT+: J1.2, J2.A15 (Pin_15), J2.A16 (Pin_16)
- new net FSPI_MISO: J2.B4 (Pin_4)
- new net FSPI_SCK: J2.B2 (Pin_2)
- new net GROUND_ETH_VENT: J4.5
- new net GROUND_LOX_VENT: J4.6
- new net LOX_VENT+: J1.1, J2.A11 (Pin_11), J2.A12 (Pin_12)
- new net REDS_ETH: J4.13 (P13)
- new net REDS_GND: J4.12 (P12)
- new net REDS_LOX_VENT: J4.14 (P14)
- no-connect marks 33 -> 31
Other:
- moved on the sheet: J2A
