File: flight-module/Connector-board/_autosave-Connector-board.kicad_pcb (KiCad board)
At the start: 4 copper layers, 0 parts

Commit message: Commit changes to the Connector
Routing:
- net (no net): track 0.00 -> 5273.3 mm
- net 12V: track 363.1 -> 0.00 mm
- net HX5: track 297.7 -> 0.00 mm
- net 3.3V: track 293.4 -> 0.00 mm
- net HX CLK: track 262.4 -> 0.00 mm
- net HX3: track 262.4 -> 0.00 mm
- net SD, TC MISO: track 262.3 -> 0.00 mm
- net HX7: track 241.6 -> 0.00 mm
- net HX1: track 237.9 -> 0.00 mm
- net HX6: track 236.2 -> 0.00 mm
- net HX8: track 233.8 -> 0.00 mm
- net SD, TC CLK: track 228.3 -> 0.00 mm
- net TC CLK: track 223.3 -> 0.00 mm
- net TC MISO: track 215.4 -> 0.00 mm
- net 5V: track 211.1 -> 0.00 mm
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