File: flight-module/Connector-board/max31855_breakout.kicad_sch (KiCad schematic)
At the start: 6 parts, among them U2 MAX31855KASA

Commit message: Commit changes to the Connector
Parts:
- renumbered C3 to C5, C4 to C6, R2 to R4
