File: flight-module/Connector-board/_autosave-Connector-board.kicad_sch (KiCad schematic)
At the start: 15 parts, among them J2 Stack_Shape

Commit message: completed routing
Parts:
- renumbered 4TC_DSUB to 4TC_DSUB1, GND_DSUB to GND_DSUB1, J2 to J1, PT_DSUB to PT_DSUB1, SOLENOIDS_DSUB to SOLENOIDS_DSUB1
Connections:
- net GND: now also J1.B17 (Pin_17), J1.B5 (Pin_5), J1.B9 (Pin_9)
Changed lines of the file:
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@@
   (junction (at 24.384 77.343) (diameter 0) (color 0 0 0 0)
   )
-  (junction (at 115.697 165.1) (diameter 0) (color 0 0 0 0)
-  )
   (junction (at 170.942 85.344) (diameter 0) (color 0 0 0 0)
   )
@@
   (junction (at 176.276 56.896) (diameter 0) (color 0 0 0 0)
   )
+  (junction (at 115.951 165.1) (diameter 0) (color 0 0 0 0)
+  )
   (junction (at 116.078 175.26) (diameter 0) (color 0 0 0 0)
   )
@@
   )
   (junction (at 75.692 154.432) (diameter 0) (color 0 0 0 0)
+  )
+  (junction (at 115.951 154.94) (diameter 0) (color 0 0 0 0)
   )
   (no_connect (at 73.406 162.052))
@@
     (stroke (width 0) (type default))
   )
-  (wire (pts (xy 115.697 165.1) (xy 124.714 165.1))
+  (wire (pts (xy 115.697 165.1) (xy 115.951 165.1))
     (stroke (width 0) (type default))
   )
@@
     (stroke (width 0) (type default))
   )
+  (wire (pts (xy 115.951 165.1) (xy 124.714 165.1))
+    (stroke (width 0) (type default))
+  )
   (wire (pts (xy 74.422 133.985) (xy 74.422 134.112))
     (stroke (width 0) (type default))
@@
     (stroke (width 0) (type default))
   )
-  (wire (pts (xy 115.697 155.067) (xy 115.697 165.1))
+  (wire (pts (xy 115.951 154.94) (xy 115.951 165.1))
     (stroke (width 0) (type default))
   )
@@
   (symbol (lib_id "Connector:DB15_Female") (at 67.056 38.354 0) (unit 1)
     (in_bom yes) (on_board yes) (dnp no)
-    (property "Reference" "GND_DSUB" (at 74.168 37.211 0)
+    (property "Reference" "GND_DSUB1" (at 74.168 37.211 0)
       (effects (font (size 1.27 1.27)) (justify right))
     )
@@
       (project "Connector-board"
         (path "/9e0a4b39-2b30-4bec-9684-92acf902e3a8"
-          (reference "GND_DSUB") (unit 1)
+          (reference "GND_DSUB1") (unit 1)
         )
       )
@@
   (symbol (lib_id "Connector:DE9_Receptacle") (at 76.962 94.615 0) (unit 1)
     (in_bom yes) (on_board yes) (dnp no) (fields_autoplaced)
-    (property "Reference" "4TC_DSUB" (at 82.55 93.345 0)
+    (property "Reference" "4TC_DSUB1" (at 82.55 93.345 0)
       (effects (font (size 1.27 1.27)) (justify left))
     )
@@
       (project "Connector-board"
         (path "/9e0a4b39-2b30-4bec-9684-92acf902e3a8"
-          (reference "4TC_DSUB") (unit 1)
+          (reference "4TC_DSUB1") (unit 1)
         )
       )
@@
   (symbol (lib_id "Connector:DE9_Receptacle") (at 39.751 79.883 0) (unit 1)
     (in_bom yes) (on_board yes) (dnp no) (fields_autoplaced)
-    (property "Reference" "SOLENOIDS_DSUB" (at 44.45 78.613 0)
+    (property "Reference" "SOLENOIDS_DSUB1" (at 44.45 78.613 0)
       (effects (font (size 1.27 1.27)) (justify left))
     )
@@
       (project "Connector-board"
         (path "/9e0a4b39-2b30-4bec-9684-92acf902e3a8"
-          (reference "SOLENOIDS_DSUB") (unit 1)
+          (reference "SOLENOIDS_DSUB1") (unit 1)
         )
       )
@@
   (symbol (lib_id "Connector:DB25_Receptacle") (at 106.68 57.15 0) (unit 1)
     (in_bom yes) (on_board yes) (dnp no) (fields_autoplaced)
-    (property "Reference" "PT_DSUB" (at 111.76 55.88 0)
+    (property "Reference" "PT_DSUB1" (at 111.76 55.88 0)
       (effects (font (size 1.27 1.27)) (justify left))
     )
@@
       (project "Connector-board"
         (path "/9e0a4b39-2b30-4bec-9684-92acf902e3a8"
-          (reference "PT_DSUB") (unit 1)
+          (reference "PT_DSUB1") (unit 1)
         )
       )
@@
   (symbol (lib_id "Stack_Shape:Stack_Shape") (at 56.896 160.782 0) (unit 1)
     (in_bom yes) (on_board yes) (dnp no)
-    (property "Reference" "J2" (at 55.6259 127.8721 0)
+    (property "Reference" "J1" (at 55.6259 127.8721 0)
       (effects (font (size 1.27 1.27)))
     )
@@
       (project "Connector-board"
         (path "/9e0a4b39-2b30-4bec-9684-92acf902e3a8"
-          (reference "J2") (unit 1)
+          (reference "J1") (unit 1)
         )
       )
@@
   (symbol (lib_id "Stack_Shape:Stack_Shape") (at 143.764 161.29 0) (unit 2)
     (in_bom yes) (on_board yes) (dnp no) (fields_autoplaced)
-    (property "Reference" "J2" (at 142.494 128.3802 0)
+    (property "Reference" "J1" (at 142.494 128.3802 0)
       (effects (font (size 1.27 1.27)))
     )
@@
       (project "Connector-board"
         (path "/9e0a4b39-2b30-4bec-9684-92acf902e3a8"
-          (reference "J2") (unit 2)
-        )
-      )
+          (reference "J1") (unit 2)
+        )
+      )
