File: TC-board/TC-board.kicad_pcb (KiCad board)
At the start: 2 copper layers, 63.5 x 63.6 mm, 13 parts, among them J1 DB15_Female, J2 PCIE-LP-01-01-F-DV-A-TR, J3 Conn_01x08_Male, J4 Conn_01x02_Male, J5 Conn_01x02_Male

Commit message: Updates to traces in TC board and updates PCIe connector
Parts:
- J2: value PCIE-LP-01-01-F-DV-A-TR -> PCIe_x16; footprint Connector_PCBEdge:BUS_PCIexpress_x1 -> PCIe_16x_DAQ:Custom-16x-PCIELock; moved to B.Cu
- moved J2 20.2 mm to (164.5, 112.1), turned to 180 degrees
Connections:
- A1 pad 7: /SPI1_MISO -> SPI1_MISO
- A2 pad 7: /SPI1_MISO -> SPI1_MISO
- A3 pad 7: /SPI1_MISO -> SPI1_MISO
- A4 pad 7: /SPI0_MISO -> SPI0_MISO
- J2 pad A10: unconnected-(J2-PadA10) -> +3.3V
- J2 pad A11: /CS4 -> unconnected-(J2-PWRGD-PadA11)
- J2 pad A18: unconnected-(J2-PadA18) -> GND
- J2 pad A2: unconnected-(J2-PadA2) -> unconnected-(J2-+12V-PadA2)
- J2 pad A3: GND -> unconnected-(J2-+12V-PadA2)
- J2 pad A4: /SPI1_SCK -> GND
- J2 pad A5: /SPI1_MISO -> unconnected-(J2-5V-PadA5)
- J2 pad A6: GND -> unconnected-(J2-5V-PadA5)
- J2 pad A7: unconnected-(J2-PadA7) -> GND
- J2 pad A8: unconnected-(J2-PadA8) -> +3.3V
- J2 pad A9: unconnected-(J2-PadA9) -> +3.3V
- J2 pad B1: /SPI0_SCK -> unconnected-(J2-+12V-PadA2)
- J2 pad B10: /CS2 -> +3.3V
- J2 pad B11: /CS3 -> unconnected-(J2-~{WAKE}-PadB11)
- J2 pad B12: GND -> unconnected-(J2-RSVD-PadB12)
- J2 pad B13: +3.3V -> GND
- J2 pad B14: +3.3V -> unconnected-(J2-I2C_SCL-PadB14)
- J2 pad B15: GND -> unconnected-(J2-I2C_SDA-PadB15)
- J2 pad B16: unconnected-(J2-PadB16) -> GND
- J2 pad B18: unconnected-(J2-PadB18) -> GND
- J2 pad B2: /SPI0_MISO -> unconnected-(J2-+12V-PadA2)
- J2 pad B3: GND -> unconnected-(J2-+12V-PadA2)
- J2 pad B4: unconnected-(J2-PadB4) -> GND
- J2 pad B5: unconnected-(J2-PadB5) -> unconnected-(J2-5V-PadA5)
- J2 pad B6: unconnected-(J2-PadB6) -> unconnected-(J2-5V-PadA5)
- J2 pad B7: unconnected-(J2-PadB7) -> GND
- J2 pad B8: unconnected-(J2-PadB8) -> +3.3V
- J2 pad B9: /CS1 -> +3.3V
- J4 pad 2: /SPI0_MISO -> SPI0_MISO
- J5 pad 2: /SPI1_MISO -> SPI1_MISO
- JP1 pad 2: /CS1 -> CS1
- JP2 pad 2: /CS2 -> CS2
- JP3 pad 2: /CS3 -> CS3
- JP4 pad 2: /CS4 -> CS4
Routing:
- net SPI1_MISO: track 0.00 -> 147.9 mm, vias 0 -> 4
- net /SPI1_MISO: track 124.2 -> 0.00 mm, vias 3 -> 0
- net CS3: track 0.00 -> 86.2 mm, vias 0 -> 6
- net CS4: track 0.00 -> 75.7 mm, vias 0 -> 4
- net GND: track 150.2 -> 75.4 mm, vias 8 -> 4
- net CS2: track 0.00 -> 56.9 mm, vias 0 -> 7
- net SPI0_MISO: track 0.00 -> 56.4 mm, vias 0 -> 4
- net /CS3: track 55.4 -> 0.00 mm, vias 4 -> 0
- net /CS1: track 47.6 -> 0.00 mm, vias 4 -> 0
- net /SPI0_MISO: track 44.4 -> 0.00 mm, vias 2 -> 0
- net /CS4: track 41.0 -> 0.00 mm, vias 3 -> 0
- net CS1: track 0.00 -> 34.9 mm, vias 0 -> 4
- net /CS2: track 28.9 -> 0.00 mm, vias 4 -> 0
- net /SPI1_SCK: track 105.7 -> 83.2 mm
- net +3.3V: track 155.3 -> 167.8 mm, vias 4 -> 5
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Other:
- board size 63.5 x 63.6 mm -> 100.6 x 64.1 mm
