File: CORE_BOARD_NEW/Core-Board.kicad_pcb (KiCad board)
At the start: 4 copper layers, 127 x 95.2 mm, 22 parts, among them J1 POWER, J1 Pin Jumper, J2 Bus_PCI_Express_x16, J3 ESP32-DEVKITC-32D, J3 XT60-M, J4 Conn_01x19_Male, J5 Conn_01x19_Male, U1 AZ1117IH-3.3TRG1, U2 AZ1117IH-5TRG1, U3 74HC4050D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

Commit message: fixed drc errors
Routing:
- net GND: track 61.0 -> 99.3 mm, vias 12 -> 20
- net HX CLK: track 54.0 -> 57.5 mm
- net HX6: track 46.0 -> 46.7 mm
- net SPI0 MISO: track 111.9 -> 112.5 mm
Other:
- board text added: "Power DAQ LE2 Hotfire 2024"
- board text removed: "Ground DAQ 2 LE2 Hotfire 2023"
