File: flight-module/Core-board/Core-board.kicad_sch (KiCad schematic)
At the start: 28 parts, among them J10 Pin Jumper, J13 Conn_01x08_Male, J18 Conn_01x02_Male, J19 Conn_01x02_Male, J20 Conn_01x02_Male, J6 ESP32-DEVKITC-32D, J7 Conn_01x19_Male, J9 Conn_01x19_Male, SW1 SW_SPST, U2 74HC4050D, U3 XTSD04GLGEAG, U5 PCF8575DW

Commit message: skeleton for connector board
Parts:
- added J? (x2): Stack_Shape, symbol Stack_Shape:Stack_Shape
Other:
- moved on the sheet: J13, J18, J19, J20, J6, J7, J9, R2, R4, R5, R6, R?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

Commit message: worked on core-board schematic. Not done.
Parts:
- removed R? (x6): 100kΩ, Resistor_SMD:R_0603_1608Metric, symbol Device:R_Small
- removed R? (x6): 2kΩ, Resistor_SMD:R_0603_1608Metric, symbol Device:R_Small
- added R14, R15, R16, R20, R21, R22: 100kΩ, Resistor_SMD:R_0603_1608Metric, symbol Device:R_Small
- added R17, R18, R19, R23, R24, R25: 2kΩ, Resistor_SMD:R_0603_1608Metric, symbol Device:R_Small
Connections:
- net HX2_A+: now also R20.1
- net HX2_E-: now also R23.1
- net HX3_A+: now also R16.1
- net HX3_E-: now also R19.1
- net HX4_A+: now also R21.1
- net HX4_E-: now also R24.1
- net HX5_A+: now also R15.1
- net HX5_E-: now also R18.1
- net HX6_A+: now also R22.1
- net HX6_E-: now also R25.1
- net HX711 1/A+: now also R14.2, R17.2
- net HX711 1/A-: now also R17.1
- net HX711 2/A+: now also R20.2, R23.2
- net HX711 3/A+: now also R16.2, R19.2
- net HX711 4/A+: now also R21.2, R24.2
- net HX711 5/A+: now also R15.2, R18.2
- net HX711 6/A+: now also R22.2, R25.2
Other:
- added sheet ESP32-Breakout (ESP32-Breakout.kicad_sch)

Commit message: Updated core-board
Parts:
- removed J10: Pin Jumper, Connector_PinHeader_2.54mm:PinHeader_1x02_P2.54mm_Vertical, symbol Connector:Conn_01x02_Male
- removed J13: Conn_01x08_Male, Connector_PinHeader_2.54mm:PinHeader_1x08_P2.54mm_Vertical, symbol Connector:Conn_01x08_Male
- removed J18, J19, J20: Conn_01x02_Male, Connector_PinHeader_2.54mm:PinHeader_1x02_P2.54mm_Vertical, symbol Connector:Conn_01x02_Male
- removed J6: ESP32-DEVKITC-32D, Ellie_Project_Footprints:MODULE_ESP32-DEVKITC-32D, symbol ESP32:ESP32-DEVKITC-32D
- removed R2: 1k, Resistor_SMD:R_0603_1608Metric, symbol Device:R_Small
- removed R4, R5, R6: 10k, Resistor_SMD:R_0603_1608Metric, symbol Device:R_Small
- removed SW1: SW_SPST, Button_Switch_THT:SW_PUSH_6mm, symbol Switch:SW_SPST
- removed U5: PCF8575DW, PCF8575DW:SOIC127P1030X265-24N, symbol PCF8575DW:PCF8575DW
Connections:
- net 5V is gone; now on net HX1_DT: J7.1 (Pin_1)
- net EN is gone; now on net EX1: J7.18 (Pin_18)
- net HX CLK is gone; now on net SPI_CLK: J7.9 (Pin_9)
- net HX1 is gone; now on net I2C_SCL: J7.17 (Pin_17)
- net HX2 is gone; now on net I2C_SDA: J7.16 (Pin_16)
- net HX4 is gone; now on net TC4_CS: J7.14 (Pin_14)
- net HX5 is gone; now on net TC3_CS: J7.13 (Pin_13)
- net HX6 is gone; now on net TC2_CS: J7.12 (Pin_12)
- net HX7 is gone; now on net TC1_CS: J7.11 (Pin_11)
- net HX711 1/A- is gone; now on net HX1_E-: R17.1
- net HX8 is gone; now on net SD_CS: J7.10 (Pin_10)
- net TC CLK is gone; now on net SPI_MISO: J7.8 (Pin_8)
- net TC MISO is gone; now on net HX5_DT: J7.5 (Pin_5)
- net +3.3V: now also J?.A1 (Pin_1), J?.A2 (Pin_2), U2.1 (VCC), U3.8 (VDD)
- net +5V: now also J?.A5 (Pin_5), J?.A6 (Pin_6), J?.A7 (Pin_7), J?.A8 (Pin_8)
- net GND: now also J?.B14 (Pin_14), J?.B17 (Pin_17), J?.B20 (Pin_20), J?.B25 (Pin_25), J?.B26 (Pin_26), J?.B33 (Pin_33), J?.B34 (Pin_34), J?.B5 (Pin_5), J?.B8 (Pin_8), J?.B9 (Pin_9); no longer J7.6 (Pin_6), J9.1 (Pin_1), J9.7 (Pin_7)
- net HX1_E+: now also J?.B11 (Pin_11)
- net HX2_A+: now also J?.B23 (Pin_23)
- net HX2_DT: now also J7.2 (Pin_2)
- net HX2_E+: now also J?.B19 (Pin_19)
- net HX2_E-: now also J?.B21 (Pin_21)
- net HX3_A+: now also J?.B31 (Pin_31)
- net HX3_DT: now also J7.3 (Pin_3)
- net HX3_E+: now also J?.B27 (Pin_27)
- net HX3_E-: now also J?.B29 (Pin_29)
- net HX4_A+: now also J?.B39 (Pin_39)
- net HX4_DT: now also J7.4 (Pin_4)
- net HX4_E+: now also J?.B35 (Pin_35)
- net HX4_E-: now also J?.B37 (Pin_37)
- net HX5_A+: now also J?.B32 (Pin_32)
- net HX5_E+: now also J?.B28 (Pin_28)
- net HX5_E-: now also J?.B30 (Pin_30)
- net HX6_A+: now also J?.B40 (Pin_40)
- net HX6_DT: now also J7.6 (Pin_6)
- net HX6_E+: now also J?.B36 (Pin_36)
- net HX6_E-: now also J?.B38 (Pin_38)
- net HX1_A+: now reaches R14.1
- net HX1_A+: now also J?.B15 (Pin_15)
- net SPI_MOSI: now reaches J7.7 (Pin_7)
- net SPI_MOSI: now also J?.B6 (Pin_6), U2.3 (1A)
- net I2C_SDA: now reaches J?.B1 (Pin_1)
- net TC1_CS: now reaches J?.B10 (Pin_10)
- net TC2_CS: now reaches J?.B12 (Pin_12)
- net HX1_E-: now reaches J?.B13 (Pin_13)
- net TC3_CS: now reaches J?.B16 (Pin_16)
- net TC4_CS: now reaches J?.B18 (Pin_18)
- net SPI_CLK: now reaches J?.B2 (Pin_2)
- net SPI_CLK: now also U2.5 (2A)
- net EX2: now reaches J?.B22 (Pin_22)
- net EX2: now also J7.19 (Pin_19)
- net EX3: now reaches J?.B24 (Pin_24)
- net I2C_SCL: now reaches J?.B3 (Pin_3)
- net SPI_MISO: now reaches J?.B4 (Pin_4)
- net SPI_MISO: now also U3.6 (SD0/DO)
- net EX1: now reaches J?.B7 (Pin_7)
- net SD_CS_BUF: now reaches U3.2 (SD3/~{CS})
- net SD_CS_BUF: now also U2.6 (3Y)
- net SD_CS: now reaches U2.7 (3A)
- removed net 3.3V: J7.19 (Pin_19), U2.1 (VCC), U3.8 (VDD)
- net HX3 renamed SPI_CS0
- net I2C SCL: no longer names the net of J9.3 (Pin_3)
- net I2C SDA: no longer names the net of J9.6 (Pin_6)
- net SD CLK: no longer names the net of J9.9 (Pin_9)
- net SD CLK: no longer U2.5 (2A)
- net SD CLK_3.3 renamed SPI_CLK_BUF
- net SD CS: no longer names the net of J9.10 (Pin_10)
- net SD CS: no longer U2.9 (4A)
- net SD CS_3.3: no longer names the net of U2.10 (4Y)
- net SD MISO: no longer names the net of J9.2 (Pin_2)
- net SD MISO: no longer U3.6 (SD0/DO)
- net SD MOSI: no longer names the net of J9.8 (Pin_8)
- net SD MOSI: no longer U2.3 (1A)
- net SD MOSI_3.3 renamed SPI_MOSI_BUF
- net SERIAL_RX: no longer names the net of J9.12 (Pin_12)
- net SERIAL_TX: no longer names the net of J9.13 (Pin_13)
- net TC MOSI: no longer names the net of J9.11 (Pin_11)
- no-connect marks 41 -> 47
Other:
- sheet ESP32-Breakout renamed ESP32-S3-WROOM-1-Breakout
- sheet ESP32-S3-WROOM-1-Breakout ports: added IO1, IO10, IO11, IO12, IO13, IO14, IO15, IO16, IO17, IO18, IO2, IO21, IO38, IO39, IO4, IO40, IO41, IO42, IO47, IO48, IO5, IO6, IO7, IO8, IO9; removed none
- note removed: "ESP32"
- moved on the sheet: J7, J9, J?A, J?B, R14, R15, R16, R17, R18, R19, R20, R21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

Commit message: update on flight pcbs
Parts:
- removed J9: Conn_01x19_Male, Connector_PinHeader_2.54mm:PinHeader_1x19_P2.54mm_Vertical, symbol Connector:Conn_01x19_Male
- gave numbers to parts that had none: 1
Connections:
- net EX1: now also J7.14 (Pin_14); no longer J7.18 (Pin_18)
- net EX2: now also J7.15 (Pin_15); no longer J7.19 (Pin_19)
- net EX3: now also J7.16 (Pin_16)
- net I2C_SCL: now also J7.13 (Pin_13); no longer J7.17 (Pin_17)
- net I2C_SDA: now also J7.12 (Pin_12); no longer J7.16 (Pin_16)
- net SPI_CS0: now also J7.11 (Pin_11); no longer J7.15 (Pin_15)
- net TC1_CS: no longer J7.11 (Pin_11)
- net TC2_CS: no longer J7.12 (Pin_12)
- net TC3_CS: no longer J7.13 (Pin_13)
- net TC4_CS: no longer J7.14 (Pin_14)
- no-connect marks 47 -> 49
Other:
- moved on the sheet: J7

Commit message: Progress on core board.
Parts:
- removed J7: Conn_01x19_Male, Connector_PinHeader_2.54mm:PinHeader_1x19_P2.54mm_Vertical, symbol Connector:Conn_01x19_Male
- added J4: Conn_01x06_Pin, Connector_PinHeader_2.54mm:PinHeader_1x06_P2.54mm_Vertical, symbol Connector:Conn_01x06_Pin
- J1: footprint (none) -> Stack_Shape:Stack_Shape
- renumbered R14 to R1, R23 to R10, R24 to R11, R25 to R12, R15 to R2, R16 to R3, R17 to R4, R18 to R5, R19 to R6, R20 to R7, R21 to R8, R22 to R9, U3 to U7, U2 to U8
Connections:
- net +3.3V: now also J4.5 (Pin_5)
- net GND: now also J1.A10 (Pin_10), J1.A13 (Pin_13), J1.A14 (Pin_14), J1.A17 (Pin_17), J1.A18 (Pin_18), J1.A21 (Pin_21), J1.A22 (Pin_22), J1.A25 (Pin_25), J1.A26 (Pin_26), J1.A3 (Pin_3), J1.A4 (Pin_4), J1.A9 (Pin_9), J1.B18 (Pin_18), J4.6 (Pin_6); no longer J1.B14 (Pin_14), J1.B20 (Pin_20)
- net SD_CS_BUF: now also J4.4 (Pin_4)
- net SPI_CLK_BUF: now also J4.3 (Pin_3)
- net SPI_MISO: now also J4.2 (Pin_2)
- net SPI_MOSI_BUF: now also J4.1 (Pin_1)
- net TC3_CS: now also J1.B14 (Pin_14); no longer J1.B16 (Pin_16)
- net TC4_CS: now also J1.B16 (Pin_16); no longer J1.B18 (Pin_18)
- net EX1 renamed PYRO1EN
- net EX2 renamed PYRO3EN
- net EX3 renamed PYRO4EN
- new net PYRO2EN: J1.B20 (Pin_20)
- no-connect marks 49 -> 34
Other:
- moved on the sheet: J1A, J1B, R1, R10, R11, R12, R2, R3, R4, R5, R6, R7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
