File: flight-module/Core-board/Core-board.kicad_pcb (KiCad board)
At the start: 4 copper layers, 141.7 x 134.1 mm, 96 parts, among them J1 Stack_Shape, J2 Conn_01x03_Pin, J3 USB_B_Micro, J4 Conn_01x06_Pin, J5 Conn_01x03_Pin, J6 Conn_01x03_Pin, J7 Conn_01x03_Pin, J8 Conn_01x03_Pin, J9 Conn_01x03_Pin, Q1 MMBT4403LT3G, Q2 MMBT4403LT3G, Q3 MMBT4403LT3G, Q4 MMBT4403LT3G, Q5 MMBT4403LT3G, Q6 MMBT4403LT3G, SW1 SW_MEC_5E, SW2 SW_MEC_5E, U1 HX711, U10 ESP32-S3-WROOM-1-N16R2, U2 HX711, U3 HX711, U4 HX711, U5 HX711, U6 HX711, U7 XTSD04GLGEAG, U8 74HC4050D, U9 AZ1084-3.3

Commit message: Finished flight-core.
Parts:
- removed R10, R11, R12, R5, R6: 2kΩ, Resistor_SMD:R_0603_1608Metric
- removed R2, R3, R7, R8, R9: 100kΩ, Resistor_SMD:R_0603_1608Metric
- added G***: LOGO, star:star_8x7, F.Cu at (149.9, 61.8)
- added R39: 100kΩ, Resistor_SMD:R_0603_1608Metric, F.Cu at (166.3, 116.6)
- added R40: 2kΩ, Resistor_SMD:R_0603_1608Metric, F.Cu at (162.9, 117.3)
- added R41: 100kΩ, Resistor_SMD:R_0603_1608Metric, F.Cu at (109.2, 118.6)
- added R42: 2kΩ, Resistor_SMD:R_0603_1608Metric, F.Cu at (105.8, 119.3)
- added R43: 100kΩ, Resistor_SMD:R_0603_1608Metric, F.Cu at (137.0, 126.0)
- added R44: 2kΩ, Resistor_SMD:R_0603_1608Metric, F.Cu at (133.6, 126.7)
- added R45: 100kΩ, Resistor_SMD:R_0603_1608Metric, F.Cu at (166.3, 91.2)
- added R46: 2kΩ, Resistor_SMD:R_0603_1608Metric, F.Cu at (162.9, 92.0)
- added R47: 100kΩ, Resistor_SMD:R_0603_1608Metric, F.Cu at (138.3, 98.8)
- added R48: 2kΩ, Resistor_SMD:R_0603_1608Metric, F.Cu at (134.9, 99.5)
- moved U4 308.2 mm to (92.7, 124.2), turned to 180 degrees
- moved Q3 301.9 mm to (99.9, 132.1)
- moved C14 300.5 mm to (94.4, 131.8), turned to 180 degrees
- moved R25 300.3 mm to (99.5, 126.0), turned to 180 degrees
- moved C15 300.0 mm to (98.9, 119.4), turned to 90 degrees
- moved C16 299.6 mm to (98.9, 123.1), turned to 90 degrees
- moved J6 299.2 mm to (108.7, 130.3), turned to 180 degrees
- moved R23 298.3 mm to (102.3, 118.6)
- moved R24 298.3 mm to (102.3, 121.1)
- moved R26 297.4 mm to (103.1, 126.9), turned to 90 degrees
- moved C13 295.8 mm to (99.5, 128.2), turned to 180 degrees
- moved U6 285.2 mm to (149.7, 122.2), turned to 180 degrees
- moved U2 279.0 mm to (121.7, 104.4), turned to 180 degrees
- moved Q6 270.5 mm to (128.9, 112.3)
- moved C26 270.0 mm to (123.5, 112.0), turned to 180 degrees
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Connections:
- J2 pad 3: /HX711 6/A+ -> /HX6_A+
- J5 pad 3: /HX711 1/A+ -> /HX1_A+
- J6 pad 3: /HX711 4/A+ -> /HX4_A+
- J7 pad 3: /HX711 5/A+ -> /HX5_A+
- J8 pad 3: /HX711 3/A+ -> /HX3_A+
- J9 pad 3: /HX711 2/A+ -> /HX2_A+
- R1 pad 2: /HX711 1/A+ -> Net-(R1-Pad2)
- R13 pad 2: /HX711 6/A+ -> Net-(R13-Pad2)
- R17 pad 2: /HX711 1/A+ -> Net-(R1-Pad2)
- R23 pad 2: /HX711 4/A+ -> Net-(R23-Pad2)
- R27 pad 2: /HX711 5/A+ -> Net-(R27-Pad2)
- R31 pad 2: /HX711 3/A+ -> Net-(R31-Pad2)
- R35 pad 2: /HX711 2/A+ -> Net-(R35-Pad2)
- R4 pad 2: /HX711 1/A+ -> Net-(R1-Pad2)
Routing:
- net +3.3V: track 1.27 -> 395.0 mm, vias 0 -> 5
- net /HX_CLK: track 0.00 -> 225.2 mm, vias 0 -> 8
- net GND: track 28.7 -> 246.8 mm, vias 3 -> 28
- net /HX4_E+: track 0.00 -> 101.9 mm
- net /TC2_CS: track 0.00 -> 101.8 mm, vias 0 -> 1
- net /TC3_CS: track 0.00 -> 101.0 mm, vias 0 -> 1
- net /PYRO4EN: track 0.00 -> 100.9 mm
- net /TC4_CS: track 0.00 -> 100.5 mm, vias 0 -> 1
- net /HX5_E+: track 0.00 -> 99.7 mm
- net /TC1_CS: track 0.00 -> 99.6 mm, vias 0 -> 1
- net /PYRO3EN: track 0.00 -> 96.2 mm, vias 0 -> 2
- net /SPI_MOSI: track 0.00 -> 95.8 mm, vias 0 -> 3
- net /SPI_MISO: track 0.00 -> 92.5 mm, vias 0 -> 3
- net /PYRO2EN: track 0.00 -> 91.2 mm, vias 0 -> 2
- net /HX6_DT: track 0.00 -> 86.7 mm, vias 0 -> 2
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Other:
- board text added: "3.3"
- board text added: "A+"
- board text added: "BOOT"
- board text added: "CLK"
- board text added: "CS"
- board text added: "E+"
- board text added: "E-"
- board text added: "ESP32-S3-VROOM-1"
- board text added: "Flight Module Core Board V1"
- board text added: "GND"
- board text added: "HX1"
- board text added: "HX2"
- board text added: "HX3"
- board text added: "HX4"
- board text added: "HX5"
- board text added: "HX6"
- board text added: "MISO"
- board text added: "MOSI"
- board text added: "RESET"
- board text added: "SD Card"

Commit message: Updated core board.
Parts:
- SW1, SW2: value SW_MEC_5E -> 1825910-6; footprint Button_Switch_SMD:SW_SPST_TL3305A -> 1825910-6:SW_1825910-6-4
- moved SW1 0.89 mm to (146.7, 48.2)
- moved SW2 0.70 mm to (146.4, 36.8)
- moved C9 0.58 mm to (153.6, 48.5), turned to -90 degrees
- moved C10 0.32 mm to (153.8, 35.9), turned to -90 degrees
Connections:
- C10 pad 1: /ESP32-S3-WROOM-1-Breakout/EN -> GND
- C10 pad 2: GND -> /ESP32-S3-WROOM-1-Breakout/EN
- C9 pad 1: /ESP32-S3-WROOM-1-Breakout/BOOT -> GND
- C9 pad 2: GND -> /ESP32-S3-WROOM-1-Breakout/BOOT
- SW1 pad 2: /ESP32-S3-WROOM-1-Breakout/BOOT -> GND
- SW2 pad 2: /ESP32-S3-WROOM-1-Breakout/EN -> GND
Routing:
- net /ESP32-S3-WROOM-1-Breakout/EN: track 64.1 -> 63.4 mm
- net +3.3V: track 395.0 -> 395.6 mm
- net /ESP32-S3-WROOM-1-Breakout/BOOT: track 31.6 -> 31.0 mm
- net GND: track 246.8 -> 246.3 mm, vias 28 -> 26
