File: flight-module/Core-board/Core-board.kicad_pcb (KiCad board)
At the start: 4 copper layers, 141.7 x 134.1 mm, 98 parts, among them J1 Stack_Shape, J11 10118194-0011LF, J2 Conn_01x03_Pin, J3 Probe_points, J4 Conn_01x06_Pin, J5 Conn_01x03_Pin, J6 Conn_01x03_Pin, J7 Conn_01x03_Pin, J8 Conn_01x03_Pin, J9 Conn_01x03_Pin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

Commit message: core board sd card and HX2 HX6 changes
Parts:
- removed J4: Conn_01x06_Pin, Connector_PinHeader_2.54mm:PinHeader_1x06_P2.54mm_Vertical
- removed U7: XTSD04GLGEAG, XTSD04GLGEAG:SON127P600X800X95-8N
- removed U8: 74HC4050D, 74HC4050D:SO16
- added J10: Conn_01x07_Pin, Connector_PinSocket_2.54mm:PinSocket_1x07_P2.54mm_Vertical, F.Cu at (120.8, 73.2)
Connections:
- U10 pad 31: /ESP32-S3-WROOM-1-Breakout/IO38 -> /HX2_DT
- U10 pad 32: /ESP32-S3-WROOM-1-Breakout/IO39 -> /HX6_DT
- U10 pad 5: /HX2_DT -> /ESP32-S3-WROOM-1-Breakout/IO5
- U10 pad 9: /HX6_DT -> /ESP32-S3-WROOM-1-Breakout/IO16
Routing:
- net /SD_CS_BUF: track 38.1 -> 0.00 mm, vias 1 -> 0
- net /SD_CS: track 30.7 -> 52.8 mm, vias 2 -> 3
- net /SPI_MOSI_BUF: track 20.0 -> 0.00 mm
- net /HX2_DT: track 55.0 -> 74.5 mm
- net /SPI_CLK_BUF: track 19.3 -> 0.00 mm, vias 2 -> 0
- net /SPI_MISO: track 92.5 -> 105.8 mm
- net +3.3V: track 391.0 -> 398.7 mm
- net /HX6_DT: track 86.3 -> 93.6 mm
- net /SPI_MOSI: track 95.8 -> 101.9 mm
- net /HX3_DT: track 65.4 -> 70.9 mm
- net /SPI_CLK: track 86.7 -> 90.8 mm
- net GND: track 226.0 -> 223.0 mm, vias 27 -> 91
Other:
- board text added: "Flight Module Core Board V3"
- board text removed: "3.3"
- board text removed: "CLK"
- board text removed: "CS"
- board text removed: "Flight Module Core Board V1"
- board text removed: "GND"
- board text removed: "MISO"
- board text removed: "MOSI"
- board text removed: "SD Card"
