File: flight-module/Core-board/Core-board 2.kicad_pcb (KiCad board)
At the start: 4 copper layers, 141.7 x 134.1 mm, 97 parts, among them J1 Stack_Shape, J2 Conn_01x03_Pin, J3 USB_B_Micro, J4 Conn_01x06_Pin, J5 Conn_01x03_Pin, J6 Conn_01x03_Pin, J7 Conn_01x03_Pin, J8 Conn_01x03_Pin, J9 Conn_01x03_Pin, Q1 MMBT4403LT3G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

Commit message: merge conflict fix
Parts:
- SW1, SW2: value SW_MEC_5E -> 1825910-6; footprint Button_Switch_SMD:SW_SPST_TL3305A -> 1825910-6:SW_1825910-6-4
- moved SW1 0.89 mm to (146.7, 48.2)
- moved SW2 0.70 mm to (146.4, 36.8)
- moved C9 0.58 mm to (153.6, 48.5), turned to -90 degrees
- moved C10 0.32 mm to (153.8, 35.9), turned to -90 degrees
Connections:
- SW1 pad 2: /ESP32-S3-WROOM-1-Breakout/BOOT -> GND
- SW2 pad 2: /ESP32-S3-WROOM-1-Breakout/EN -> GND
Routing:
- net /ESP32-S3-WROOM-1-Breakout/EN: track 64.1 -> 63.4 mm
- net +3.3V: track 395.0 -> 395.6 mm
- net /ESP32-S3-WROOM-1-Breakout/BOOT: track 31.6 -> 31.0 mm
- net GND: track 246.8 -> 246.3 mm, vias 28 -> 26
